File: hardware/DuploTrainController NG/DuploTrainController NG.kicad_pcb (KiCad board)
At the start: 2 copper layers, 36 x 99 mm, 16 parts, among them SW0 Speed / SHIFT, SW1 Record, SW2 Play, SW3 Stop, SW4 Water, SW5 LED Cycle, SW6 Sound Cycle, U1 ESP32-S3_SUPERMINI_SMD

Commit message: Update hardware case and PCB assets
Parts:
- C1: footprint Capacitor_THT:C_Rect_L7.0mm_W2.0mm_P5.00mm -> Capacitor_SMD:C_0805_2012Metric
- SW0: value Speed / SHIFT -> Speed / Wakeup
- moved C1 0.95 mm to (83.5, 76.5)
Other:
- board size 36 x 99 mm -> 34.1 x 99 mm
- board text added: "Duplo Train Remote Control V1.0 R. Zuehlsdorff © 2026"
Changed lines of the file:
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@@
 			)
 		)
-		(property "Datasheet" "~"
+		(property "Datasheet" ""
 			(at 0 0 90)
 			(layer "F.Fab")
@@
 			)
 		)
-		(property "Datasheet" "~"
+		(property "Datasheet" ""
 			(at 0 0 90)
 			(layer "F.Fab")
@@
 			)
 		)
-		(property "Datasheet" "~"
+		(property "Datasheet" ""
 			(at 0 0 270)
 			(layer "F.Fab")
@@
 			)
 		)
-		(property "Datasheet" "~"
+		(property "Datasheet" ""
 			(at 0 0 0)
 			(unlocked yes)
@@
 		(at 67.74 70.88 90)
 		(property "Reference" "U1"
-			(at -5.715 -13.6525 90)
+			(at -1.42 -0.04 90)
 			(layer "F.SilkS")
 			(effects
@@
 			)
 		)
-		(property "Datasheet" "~"
+		(property "Datasheet" ""
 			(at 0 0 0)
 			(unlocked yes)
@@
 			)
 		)
-		(property "Value" "Speed / SHIFT"
+		(property "Value" "Speed / Wakeup"
 			(at 7.5 11 0)
 			(layer "F.SilkS")
@@
 			)
 		)
-		(property "Datasheet" "~"
+		(property "Datasheet" ""
 			(at 0 0 0)
 			(unlocked yes)
@@
 		)
 	)
-	(footprint "Capacitor_THT:C_Rect_L7.0mm_W2.0mm_P5.00mm"
+	(footprint "Capacitor_SMD:C_0805_2012Metric"
 		(layer "F.Cu")
-		(at 82.5 76.5)
-		(descr "C, Rect series, Radial, pin pitch=5.00mm, length*width=7*2mm^2, Capacitor")
-		(tags "C Rect series Radial pin pitch 5.00mm length 7mm width 2mm Capacitor")
+		(at 83.45 76.5)
+		(descr "Capacitor SMD 0805 (2012 Metric), square (rectangular) end terminal, IPC-7351 nominal, (Body size source: IPC-SM-782 page 76, https://www.pcb-3d.com/wordpress/wp-content/uploads/ipc-sm-782a_amendment_1_and_2.pdf, https://docs.google.com/spreadsheets/d/1BsfQQcO9C6DZCsRaXUlFlo91Tg2WpOkGARC1WS5S8t0/edit?usp=sharing), generated with kicad-footprint-generator")
+		(tags "capacitor")
 		(property "Reference" "C1"
-			(at 2.5 -2.25 0)
+			(at 0 -1.68 0)
 			(layer "F.SilkS")
 			(effects
@@
 		)
 		(property "Value" "100n"
-			(at 2.5 2.25 0)
-			(layer "F.SilkS")
+			(at 0 1.68 0)
+			(layer "F.Fab")
 			(effects
 				(font
@@
 			)
 		)
-		(property "Datasheet" "~"
+		(property "Datasheet" ""
 			(at 0 0 0)
 			(layer "F.Fab")
@@
 		(sheetname "/")
 		(sheetfile "DuploTrainController NG.kicad_sch")
-		(attr through_hole)
+		(attr smd)
 		(fp_line
-			(start -1.12 -1.12)
-			(end -1.12 1.12)
+			(start -0.261252 -0.735)
+			(end 0.261252 -0.735)
 			(stroke
 				(width 0.12)
@@
 		)
 		(fp_line
-			(start -1.12 -1.12)
-			(end 6.12 -1.12)
+			(start -0.261252 0.735)
+			(end 0.261252 0.735)
 			(stroke
 				(width 0.12)
@@
 		)
 		(fp_line
-			(start -1.12 1.12)
-			(end 6.12 1.12)
+			(start -1.7 -0.98)
+			(end 1.7 -0.98)
 			(stroke
-				(width 0.12)
+				(width 0.05)
 				(type solid)
 			)
-			(layer "F.SilkS")
+			(layer "F.CrtYd")
 		)
 		(fp_line
-			(start 6.12 -1.12)
-			(end 6.12 1.12)
+			(start -1.7 0.98)
+			(end -1.7 -0.98)
 			(stroke
-				(width 0.12)
+				(width 0.05)
 				(type solid)
 			)
-			(layer "F.SilkS")
+			(layer "F.CrtYd")
 		)
-		(fp_rect
-			(start -1.25 -1.25)
-			(end 6.25 1.25)
+		(fp_line
+			(start 1.7 -0.98)
+			(end 1.7 0.98)
+			(stroke
+				(width 0.05)
+				(type solid)
+			)
+			(layer "F.CrtYd")
+		)
+		(fp_line
+			(start 1.7 0.98)
+			(end -1.7 0.98)
 			(stroke
 				(width 0.05)
 				(type solid)
 			)
-			(fill no)
 			(layer "F.CrtYd")
 		)
-		(fp_rect
-			(start -1 -1)
-			(end 6 1)
+		(fp_line
+			(start -1 -0.625)
+			(end 1 -0.625)
 			(stroke
 				(width 0.1)
 				(type solid)
 			)
-			(fill no)
 			(layer "F.Fab")
 		)
-		(pad "1" thru_hole circle
-			(at 0 0)
-			(size 1.6 1.6)
-			(drill 0.8)
-			(layers "*.Cu" "*.Mask")
-			(remove_unused_layers no)
+		(fp_line
+			(start -1 0.625)
+			(end -1 -0.625)
+			(stroke
+				(width 0.1)
+				(type solid)
+			)
+			(layer "F.Fab")
+		)
+		(fp_line
+			(start 1 -0.625)
+			(end 1 0.625)
+			(stroke
+				(width 0.1)
+				(type solid)
+			)
+			(layer "F.Fab")
+		)
+		(fp_line
+			(start 1 0.625)
+			(end -1 0.625)
+			(stroke
+				(width 0.1)
+				(type solid)
+			)
+			(layer "F.Fab")
+		)
+		(fp_text user "${REFERENCE}"
+			(at 0 0 0)
+			(layer "F.Fab")
+			(effects
+				(font
+					(size 0.5 0.5)
+					(thickness 0.08)
+				)
+			)
+		)
+		(pad "1" smd roundrect
+			(at -0.95 0)
+			(size 1 1.45)
+			(layers "F.Cu" "F.Mask" "F.Paste")
+			(roundrect_rratio 0.25)
 			(net 2 "ADC_Buttons")
 			(pintype "passive")
 		)
-		(pad "2" thru_hole circle
-			(at 5 0)
-			(size 1.6 1.6)
-			(drill 0.8)
-			(layers "*.Cu" "*.Mask")
-			(remove_unused_layers no)
+		(pad "2" smd roundrect
+			(at 0.95 0)
+			(size 1 1.45)
+			(layers "F.Cu" "F.Mask" "F.Paste")
+			(roundrect_rratio 0.25)
 			(net 1 "GND")
 			(pintype "passive")
 		)
 		(embedded_fonts no)
-		(model "${KICAD9_3DMODEL_DIR}/Capacitor_THT.3dshapes/C_Rect_L7.0mm_W2.0mm_P5.00mm.step"
+		(model "${KICAD9_3DMODEL_DIR}/Capacitor_SMD.3dshapes/C_0805_2012Metric.step"
 			(offset
 				(xyz 0 0 0)
@@
 			)
 		)
-		(property "Datasheet" "~"
+		(property "Datasheet" ""
 			(at 0 0 0)
 			(unlocked yes)
@@
 			)
 		)
-		(property "Datasheet" "~"
+		(property "Datasheet" ""
 			(at 0 0 90)
 			(layer "F.Fab")
@@
 			)
 		)
-		(property "Datasheet" "~"
+		(property "Datasheet" ""
 			(at 0 0 90)
 			(layer "F.Fab")
@@
 			)
 		)
-		(property "Datasheet" "~"
+		(property "Datasheet" ""
 			(at 0 0 90)
 			(layer "F.Fab")
@@
 			)
 		)
-		(property "Datasheet" "~"
+		(property "Datasheet" ""
 			(at 0 0 0)
 			(unlocked yes)
@@
 			)
 		)
-		(property "Datasheet" "~"
+		(property "Datasheet" ""
 			(at 0 0 0)
 			(unlocked yes)
@@
 			)
 		)
-		(property "Datasheet" "~"
+		(property "Datasheet" ""
 			(at 0 0 0)
 			(unlocked yes)
@@
 			)
 		)
-		(property "Datasheet" "~"
+		(property "Datasheet" ""
 			(at 0 0 90)
 			(layer "F.Fab")
@@
 	(gr_poly
 		(pts
-			(xy 91.5 40) (xy 91.5 139) (xy 55.5 139) (xy 55.5 76) (xy 61 76) (xy 61 66) (xy 55.5 66) (xy 55.5 40)
+			(xy 90.55 40) (xy 90.55 139) (xy 56.45 139) (xy 56.45 76) (xy 61 76) (xy 61 66) (xy 56.45 66) (xy 56.45 40)
 		)
 		(stroke
@@
 		(layer "Edge.Cuts")
 	)
+	(gr_text "Duplo Train Remote Control\nV1.0 R. Zuehlsdorff © 2026"
+		(at 87 64.5 90)
+		(layer "F.SilkS")
+		(effects
+			(font
+				(size 1 1)
+				(thickness 0.125)
+			)
+			(justify left bottom)
+		)
+	)
 	(segment
 		(start 82.5 76.5)
@@
 		(polygon
 			(pts
-				(xy 55.5 40) (xy 91.5 40) (xy 91.5 139) (xy 55.5 139) (xy 55.5 76) (xy 79.5 76) (xy 79.5 65.5) (xy 55.5 65.5)
+				(xy 56.3 40) (xy 90.65 40) (xy 90.65 139) (xy 56.15 139) (xy 56.15 76) (xy 79.5 76) (xy 79.5 65.5)
+				(xy 56.3 65.5)
 			)
 		)
