File: hardware/DuploTrainController NG/DuploTrainController NG.kicad_sch (KiCad schematic)
At the start: 16 parts, among them SW0 Speed / SHIFT, SW1 Record, SW2 Play, SW3 Stop, SW4 Water, SW5 LED Cycle, SW6 Sound Cycle, U1 ESP32-S3_SUPERMINI_SMD

Commit message: Update hardware case and PCB assets
Parts:
- C1: footprint Capacitor_THT:C_Rect_L7.0mm_W2.0mm_P5.00mm -> Capacitor_SMD:C_0805_2012Metric
- SW0: value Speed / SHIFT -> Speed / Wakeup
Other:
- note added: "3,3V if all Buttons are open"
- note added: "Duplo Train Remote Control V1.0 2026 - Controller ESP32-S3 Supermini with Battery MAnagement Chip - All buttons will be read in as ADC values - Forward and reverse spee controlled by encoder - Press of encoder button wakes up from deep sleep Layout has been modified to fit also to smaller 5x16 dot case Height of case is 5 Lego layers."
- note added: "Function R E24 in k Uadc in V delta Encoder Btn 0 Record 0,43 0,540 0,540 Play 0,62 1,066 0,527 Stop 0,91 1,555 0,489 Water 1,5 2,017 0,463 LED Cycle 3,3 2,490 0,472 Sound Cycle 13 2,969 0,480 alle offen 3,300 0,331"
- note removed: "3,3V wenn alle Schalter offen"
- note removed: "Funktion R E24 in k Uadc in V delta Encoder Btn 0 Record 0,43 0,540 0,540 Play 0,62 1,066 0,527 Stop 0,91 1,555 0,489 Water 1,5 2,017 0,463 LED Cycle 3,3 2,490 0,472 Sound Cycle 13 2,969 0,480 alle offen 3,300 0,331"
- note removed: "fernsteuerung eines Dupplozuges Controller ESP32-S3 Supermini mit Betteriemanagement Buttons werden über ein Widerstandsnetz als ADC Value eingelesen Fahrsteuerung über Encoder"
Changed lines of the file:
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@@
 		)
 	)
-	(text "fernsteuerung eines Dupplozuges \nController ESP32-S3 Supermini mit Betteriemanagement\nButtons werden über ein Widerstandsnetz als ADC Value eingelesen\nFahrsteuerung über Encoder"
-		(exclude_from_sim no)
-		(at 181.864 172.212 0)
+	(text "Duplo Train Remote Control V1.0 2026\n- Controller ESP32-S3 Supermini with Battery MAnagement Chip \n- All buttons will be read in as ADC values\n- Forward and reverse spee controlled by encoder \n- Press of encoder button wakes up from deep sleep\nLayout has been modified to fit also to smaller 5x16 dot case \nHeight of case is 5 Lego layers."
+		(exclude_from_sim no)
+		(at 181.864 173.736 0)
 		(effects
 			(font
 				(size 1.27 1.27)
+				(thickness 0.254)
+				(bold yes)
 			)
 			(justify left)
 		)
 	)
-	(text "3,3V wenn alle Schalter offen"
+	(text "3,3V if all Buttons are open"
 		(exclude_from_sim no)
 		(at 142.24 39.878 0)
@@
 		)
 	)
-	(text "Funktion		R E24 in k		Uadc in V	delta\n\nEncoder Btn						0	\nRecord				0,43		0,540		0,540\nPlay				0,62		1,066		0,527\nStop				0,91		1,555		0,489\nWater				1,5			2,017		0,463\nLED Cycle			3,3			2,490		0,472\nSound Cycle		13			2,969		0,480\nalle offen						3,300		0,331"
+	(text "Function		R E24 in k		Uadc in V	delta\n\nEncoder Btn						0	\nRecord				0,43		0,540		0,540\nPlay				0,62		1,066		0,527\nStop				0,91		1,555		0,489\nWater				1,5			2,017		0,463\nLED Cycle			3,3			2,490		0,472\nSound Cycle		13			2,969		0,480\nalle offen						3,300		0,331"
 		(exclude_from_sim no)
 		(at 34.036 108.712 0)
@@
 			)
 		)
-		(property "Footprint" "Capacitor_THT:C_Rect_L7.0mm_W2.0mm_P5.00mm"
+		(property "Footprint" "Capacitor_SMD:C_0805_2012Metric"
 			(at 147.0152 57.15 0)
 			(effects
@@
 			)
 		)
-		(property "Value" "Speed / SHIFT"
+		(property "Value" "Speed / Wakeup"
 			(at 181.102 17.272 90)
 			(effects
